File: binary_clock.kicad_sch (KiCad schematic)
At the start: 83 parts, among them J1 Conn_01x03_Pin, P1 TYPE-C-31-M-12, SW1 TS-1088-AR02016, SW2 TS-1088-AR02016, SW3 TS-1088-AR02016, SW4 TS-1088-AR02016, SW5 TIMEZONE_CHANGE, U1 RP2040, U2 W25Q32JVSS, U3 AMS1117-3.3, U4 DS3231M, U5 AT24C32_SOIC, Y1 ABM8-272-T3

Commit message: add USB netclass
Connections:
- net RP_USB_P: now reaches R1.2, U1.47 (USB_DP)
- net RP_USB_N: now reaches R2.2, U1.46 (USB_DM)
- net USB_DM renamed USB_N
- net USB_DP renamed USB_P
Other:
- moved on the sheet: R1, R2
Changed lines of the file:
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@@
 	(wire
 		(pts
-			(xy 158.75 57.15) (xy 162.56 57.15)
+			(xy 151.13 57.15) (xy 154.94 57.15)
 		)
 		(stroke
@@
 	(wire
 		(pts
-			(xy 170.18 54.61) (xy 172.72 54.61)
+			(xy 162.56 54.61) (xy 172.72 54.61)
 		)
 		(stroke
@@
 	(wire
 		(pts
-			(xy 170.18 57.15) (xy 172.72 57.15)
+			(xy 162.56 57.15) (xy 172.72 57.15)
 		)
 		(stroke
@@
 	(wire
 		(pts
-			(xy 158.75 54.61) (xy 162.56 54.61)
+			(xy 151.13 54.61) (xy 154.94 54.61)
 		)
 		(stroke
@@
 		)
 	)
+	(label "RP_USB_P"
+		(at 172.72 54.61 180)
+		(effects
+			(font
+				(size 1.27 1.27)
+			)
+			(justify right bottom)
+		)
+	)
 	(label "SCL"
 		(at 226.06 59.69 0)
@@
 		)
 	)
-	(label "USB_DP"
-		(at 158.75 54.61 180)
+	(label "USB_P"
+		(at 151.13 54.61 180)
 		(effects
 			(font
@@
 		)
 	)
-	(label "USB_DM"
-		(at 158.75 57.15 180)
+	(label "USB_N"
+		(at 151.13 57.15 180)
 		(effects
 			(font
@@
 		)
 	)
-	(label "USB_DM"
+	(label "USB_N"
 		(at 58.42 160.02 0)
 		(effects
@@
 		)
 	)
+	(label "RP_USB_N"
+		(at 172.72 57.15 180)
+		(effects
+			(font
+				(size 1.27 1.27)
+			)
+			(justify right bottom)
+		)
+	)
 	(label "SCL"
 		(at 45.72 109.22 180)
@@
 		)
 	)
-	(label "USB_DP"
+	(label "USB_P"
 		(at 58.42 165.1 0)
 		(effects
@@
 	(symbol
 		(lib_id "Device:R")
-		(at 166.37 54.61 90)
+		(at 158.75 54.61 90)
 		(unit 1)
 		(exclude_from_sim no)
@@
 		(dnp no)
 		(property "Reference" "R1"
-			(at 166.37 50.546 90)
+			(at 158.75 50.546 90)
 			(effects
 				(font
@@
 		)
 		(property "Value" "33"
-			(at 166.37 52.578 90)
+			(at 158.75 52.578 90)
 			(effects
 				(font
@@
 		)
 		(property "Footprint" "Resistor_SMD:R_0603_1608Metric"
-			(at 166.37 56.388 90)
+			(at 158.75 56.388 90)
 			(effects
 				(font
@@
 		)
 		(property "Datasheet" "~"
-			(at 166.37 54.61 0)
+			(at 158.75 54.61 0)
 			(effects
 				(font
@@
 		)
 		(property "Description" "Resistor"
-			(at 166.37 54.61 0)
+			(at 158.75 54.61 0)
 			(effects
 				(font
@@
 	(symbol
 		(lib_id "Device:R")
-		(at 166.37 57.15 90)
+		(at 158.75 57.15 90)
 		(unit 1)
 		(exclude_from_sim no)
@@
 		(dnp no)
 		(property "Reference" "R2"
-			(at 166.37 59.436 90)
+			(at 158.75 59.436 90)
 			(effects
 				(font
@@
 		)
 		(property "Value" "33"
-			(at 166.37 61.468 90)
+			(at 158.75 61.468 90)
 			(effects
 				(font
@@
 		)
 		(property "Footprint" "Resistor_SMD:R_0603_1608Metric"
-			(at 166.37 58.928 90)
+			(at 158.75 58.928 90)
 			(effects
 				(font
@@
 		)
 		(property "Datasheet" "~"
-			(at 166.37 57.15 0)
+			(at 158.75 57.15 0)
 			(effects
 				(font
@@
 		)
 		(property "Description" "Resistor"
-			(at 166.37 57.15 0)
+			(at 158.75 57.15 0)
 			(effects
 				(font
@@
 		(on_board yes)
 		(dnp no)
-		(fields_autoplaced yes)
 		(property "Reference" "U2"
-			(at 137.16 49.5299 0)
+			(at 136.906 47.752 0)
 			(effects
 				(font
@@
 		)
 		(property "Value" "W25Q32JVSS"
-			(at 137.16 52.0699 0)
+			(at 136.906 50.292 0)
 			(effects
 				(font
